Commit message: Adição de velocidade de movimentação pros motores, first_pose do braço, gripper funcional(?) na visualização.

File: src/movement/humanoid_visualization/urdf/hook.urdf (robot description, URDF)
Before this commit: robot hook, 11 links, 10 joints
Links:
- removed link GRIPPER
- added link LEFT_GRIPPER_FINGER; visual box size=0.02 0.01 0.0678
- added link RIGHT_GRIPPER_FINGER; visual box size=0.02 0.01 0.0678
Joints:
- removed joint GRIPPER_UX_joint
- added joint LEFT_GRIPPER_FINGER_joint: type prismatic, parent WRIST_UZ, child LEFT_GRIPPER_FINGER, origin xyz=0 0 0.093 rpy=0 0 0, axis 0 1 0, limit lower=0 upper=0.028 effort=1000.0 velocity=10
- added joint RIGHT_GRIPPER_FINGER_joint: type prismatic, parent WRIST_UZ, child RIGHT_GRIPPER_FINGER, origin xyz=0 0 0.093 rpy=0 0 0, axis 0 -1 0, limit lower=0 upper=0.028 effort=1000.0 velocity=10
- joint SHOULDER_UY_joint: axis 0 1 0 -> 0 -1 0
- joint WRIST_UZ_joint: origin xyz=0 0 0.02435 rpy=0 0 0 -> xyz=0 0 0.0205 rpy=0 0 0

Commit message: Inicio do desenvolvimento da IK e algumas correções.

File: src/movement/humanoid_visualization/urdf/hook.urdf (robot description, URDF)
Before this commit: robot hook, 12 links, 11 joints
Joints:
- joint SHOULDER_UY_joint: axis 0 -1 0 -> 0 1 0
